Commit message: 0704

File: my_robo_description/urdf/my_robo.xacro (robot description, xacro)
@@ -92,5 +92,5 @@
     <origin rpy="-1.5707 0 0" xyz="0 0.1425 -0.0175"/>
     <axis xyz="0 0 1"/>
-    <limit velocity="1.0" effort="8.0"/>	<!--decide mortor power-->
+    <limit velocity="1.0" effort="6.0"/>	<!--decide mortor power-->
     <dynamics damping="0.2"/>                   <!--damping of axes of mortor-->
   </joint>
@@ -121,5 +121,5 @@
     <origin rpy="1.5707 0 0" xyz="0 -0.1425 -0.0175"/>
     <axis xyz="0 0 -1"/>
-    <limit velocity="1.0" effort="8.0"/>
+    <limit velocity="1.0" effort="6.0"/>
     <dynamics damping="0.2"/>
   </joint>
@@ -325,6 +325,6 @@
  <gazebo reference="left_wheel_link">
    <selfCollide>true</selfCollide>
-    <mu1 value="8" />
-    <mu2 value="8" />
+    <mu1 value="9" />
+    <mu2 value="9" />
     <kp>500000.0</kp>
     <kd>10.0</kd>
@@ -336,6 +336,6 @@
  <gazebo reference="right_wheel_link">
    <selfCollide>true</selfCollide>
-    <mu1 value="8" />
-    <mu2 value="8" />
+    <mu1 value="9" />
+    <mu2 value="9" />
     <kp>500000.0</kp>
     <kd>10.0</kd>
@@ -392,5 +392,5 @@
        <plugin name="gazebo_ros_lidar_controller" filename="libgazebo_ros_laser.so">
     <!--  <plugin name="gazebo_ros_head_hokuyo_controller" filename="libgazebo_ros_gpu_laser.so"> -->
-          <topicName>/laserscan</topicName>
+          <topicName>/scan</topicName>
           <frameName>laser</frameName>
         </plugin>

Commit message: moving program.during Debug. Create test marker node

File: my_robo_description/urdf/my_robo.xacro (robot description, xacro)
@@ -92,5 +92,5 @@
     <origin rpy="-1.5707 0 0" xyz="0 0.1425 -0.0175"/>
     <axis xyz="0 0 1"/>
-    <limit velocity="1.0" effort="6.0"/>	<!--decide mortor power-->
+    <limit velocity="1.0" effort="5.0"/>	<!--decide mortor power-->
     <dynamics damping="0.2"/>                   <!--damping of axes of mortor-->
   </joint>
@@ -121,5 +121,5 @@
     <origin rpy="1.5707 0 0" xyz="0 -0.1425 -0.0175"/>
     <axis xyz="0 0 -1"/>
-    <limit velocity="1.0" effort="6.0"/>
+    <limit velocity="1.0" effort="5.0"/>
     <dynamics damping="0.2"/>
   </joint>

Commit message: 0724 visualization marker introduce. predictTraj and DWA success. d_U not.

File: my_robo_description/urdf/my_robo.xacro (robot description, xacro)
@@ -175,5 +175,5 @@
 		   <child link="back_caster"/>
 		<!--   <origin xyz="0 0 -0.02"/> -->
-		   <origin xyz="-0.130 0 -0.06"/>
+		   <origin xyz="-0.130 0 -0.071"/>
 		 </joint>
 		  <link name="back_caster">

Commit message: d_Uの計算を正しく行えた。Dなしでの実験が可能

File: my_robo_description/urdf/my_robo.xacro (robot description, xacro)
@@ -43,5 +43,5 @@
  </joint>
    <link name="base_link">
-    <visual>
+    <visual name = "base">
       <geometry>
         <box size="0.300 0.25 0.065"/>
@@ -72,10 +72,16 @@
       <origin xyz="-0.130 0 -0.0525"/>
     </visual>
-   <collision>
-      <geometry>
-        <box size="0.300 0.250 0.465"/>
-      </geometry>
-	<origin xyz="0 0 0.20" rpy="0 0 0"/>
+   <collision nane = "base">
+      <geometry>
+        <box size="0.300 0.250 0.065"/>
+      </geometry>
+	<origin xyz="0 0 0" rpy="0 0 0"/>
     </collision>
+    <collision nane = "body">
+       <geometry>
+         <box size="0.200 0.250 0.4"/>
+       </geometry>
+   <origin xyz="-0.05 0 0.2325" rpy="0 0 0"/>
+     </collision>
    <inertial>
     <origin xyz="-0.05 0 0.0575"/>
@@ -92,5 +98,5 @@
     <origin rpy="-1.5707 0 0" xyz="0 0.1425 -0.0175"/>
     <axis xyz="0 0 1"/>
-    <limit velocity="1.0" effort="5.0"/>	<!--decide mortor power-->
+    <limit velocity="1.0" effort="2.0"/>	<!--decide mortor power-->
     <dynamics damping="0.2"/>                   <!--damping of axes of mortor-->
   </joint>
@@ -121,5 +127,5 @@
     <origin rpy="1.5707 0 0" xyz="0 -0.1425 -0.0175"/>
     <axis xyz="0 0 -1"/>
-    <limit velocity="1.0" effort="5.0"/>
+    <limit velocity="1.0" effort="2.0"/>
     <dynamics damping="0.2"/>
   </joint>
@@ -419,5 +425,6 @@
             <type>gaussian</type>
             <mean>0.0</mean>
-            <stddev>0.007</stddev>
+            <!-- <stddev>0.007</stddev> -->
+            <stddev>0.000</stddev>
           </noise>
         </camera>

Commit message: modification of last time.

File: my_robo_description/urdf/my_robo.xacro (robot description, xacro)
@@ -83,4 +83,10 @@
        </geometry>
    <origin xyz="-0.05 0 0.2325" rpy="0 0 0"/>
+     </collision>
+    <collision nane = "bottom">
+       <geometry>
+         <box size="0.300 0.250 0.05"/>
+       </geometry>
+   <origin xyz="0 0 -0.0575" rpy="0 0 0"/>
      </collision>
    <inertial>
@@ -221,5 +227,5 @@
         <origin xyz="0 0 0" rpy="0 0 0"/>
         <geometry>
-          <cylinder radius="0.02" length="0.06" />
+          <cylinder radius="0.025" length="0.07" />
         </geometry>
       </collision>

Commit message: add kdtree implemetation. split program into added files

File: my_robo_description/urdf/my_robo.xacro (robot description, xacro)
@@ -110,5 +110,5 @@
     <visual>
       <geometry>
-        <cylinder radius="0.075" length="0.035"/>
+        <cylinder radius="0.075" length="0.03"/>
       </geometry>
       <origin xyz="0 0 0" rpy="0 0 0"/>

Commit message: 1010

File: my_robo_description/urdf/my_robo.xacro (robot description, xacro)
@@ -92,5 +92,5 @@
    <inertial>
     <origin xyz="-0.05 0 0.0575"/>
-    <mass value="6.800"/>      <!--battery1.6kg, mainRobot 5.8kg wheel 0.3kgx2 -->
+    <mass value="5.800"/>      <!--battery1.6kg, mainRobot 5.8kg wheel 0.3kgx2 -->
 	<!--calculated as collision cuboid  -->
     <inertia ixx="0.1735275" ixy="0" ixz="0" iyy="0.1579442" iyz="0" izz="0.08641667"/>

Commit message: 1031 const variableの整理 cal_obsの計算方法変更

File: my_robo_description/urdf/my_robo.xacro (robot description, xacro)
@@ -105,5 +105,5 @@
     <axis xyz="0 0 1"/>
     <limit velocity="1.0" effort="2.0"/>	<!--decide mortor power-->
-    <dynamics damping="0.2"/>                   <!--damping of axes of mortor-->
+    <dynamics damping="0.2"/>             <!--damping of axes of mortor-->
   </joint>
  <link name="left_wheel_link">
@@ -414,5 +414,5 @@
     <gazebo reference="camera">
       <sensor type="depth" name="Kinectv2">
-	<always_on>true</always_on>
+	      <always_on>true</always_on>
         <update_rate>30.0</update_rate>
         <camera name="Kinectv2">
@@ -462,5 +462,5 @@
         <pointCloudTopicName>/camera/depth/points</pointCloudTopicName>
         <pointCloudCutoff>0.4</pointCloudCutoff>
-	<pointCloudCutoffMax>3.0</pointCloudCutoffMax>
+      	<pointCloudCutoffMax>3.0</pointCloudCutoffMax>
         <distortionK1>0.00000001</distortionK1>
         <distortionK2>0.00000001</distortionK2>

Commit message: actor collision

File: my_robo_description/urdf/my_robo.xacro (robot description, xacro)
@@ -239,5 +239,5 @@
    <parent link="laser_link"/>
    <child link="laser"/>
-   <origin xyz="0.025 0 0"/>
+   <origin xyz="0.025 0 0.75"/>
  </joint>
 <link name="laser"/>
@@ -477,4 +477,5 @@
       </plugin>
       </sensor>
+    <allow_auto_disable>0</allow_auto_disable>
     </gazebo>
 </robot>

Commit message: collision設定の変更

File: my_robo_description/urdf/my_robo.xacro (robot description, xacro)
@@ -239,5 +239,5 @@
    <parent link="laser_link"/>
    <child link="laser"/>
-   <origin xyz="0.025 0 0.75"/>
+   <origin xyz="0.025 0 0"/>
  </joint>
 <link name="laser"/>
@@ -479,3 +479,9 @@
     <allow_auto_disable>0</allow_auto_disable>
     </gazebo>
+  <!-- <xacro:arg name="gpu" default="false"/>
+  <xacro:property name="gpu" value="$(arg gpu)" />
+  <xacro:include filename="$(find velodyne_description)/urdf/VLP-16.urdf.xacro"/>
+  <VLP-16 parent="laser" name="velodyne" topic="/velodyne_points" hz="5" samples="440" gpu="${gpu}">
+    <origin xyz="0 0 0.3" rpy="0 0 0" />
+  </VLP-16> -->
 </robot>

Commit message: 公開に向けたファイルの整理

File: my_robo_description/urdf/my_robo.xacro (robot description, xacro)
@@ -267,8 +267,8 @@
 	  <joint name="camera_joint" type="fixed">
 	   <parent link="camera_link"/>
-	   <child link="camera"/>
+	   <child link="openni_camera"/>
 	   <origin xyz="0.0325 0 0" rpy="0 0 0"/>
 	  </joint>
-	  <link name="camera"/>
+	  <link name="openni_camera"/>
  <!-- ===============  Transmission =============== -->
  <transmission name="left_wheel_trans">
@@ -413,5 +413,5 @@
 <!--CAMERA-->
 <!-- parameter reference https://vision.in.tum.de/data/datasets/rgbd-dataset/file_formats -->
-    <gazebo reference="camera">
+    <gazebo reference="openni_camera">
       <sensor type="depth" name="Kinectv1">
 	      <always_on>true</always_on>
@@ -457,5 +457,5 @@
         <updateRate>0.0</updateRate>
         <cameraName>kinect_v1</cameraName>
-        <frameName>camera</frameName>
+        <frameName>openni_camera</frameName>
         <imageTopicName>/camera/rgb/image_color</imageTopicName>
         <cameraInfoTopicName>/camera/rgb/camera_info</cameraInfoTopicName>
